File: board_zynq7ext/vllink_zynq7ext.kicad_sch (KiCad schematic)
At the start: 71 parts, among them J1 Connect_J1, J10 Connect_J10, J11 Connect_J11, J12 Connect_J12, J13 Connect_J13, J14 Connect_J14, J15 IF_Xilinx14P, J16 USB_C_Receptacle_USB2.0, J17 Conn_02x05_Odd_Even, J18 Logic_Any, J19 USB_A, J2 IF_Vllink10P, J3 Connect_J3, J4 Connect_J4, J5 Connect_J5, J6 IF_Altera10P_2P00, J7 Connect_J7, J8 IF_Altera10P_2P54, J9 USB_C_Receptacle_USB2.0, U1 PW6606, U2 SN74AVC4T245PW, U3 SN74AVC4T245PW, U4 SN74AVC4T245PW, U5 SN74AVC4T245PW

Commit message: fix
Connections:
- net NET1_MX1-: now also NET1.6; no longer NET1.4
- net NET1_MX2+: now also NET1.4; no longer NET1.5
- net NET1_MX2-: now also NET1.5; no longer NET1.6
- net NET2_MX1-: now also NET2.6; no longer NET2.4
- net NET2_MX2+: now also NET2.4; no longer NET2.5
- net NET2_MX2-: now also NET2.5; no longer NET2.6
Changed lines of the file:
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@@
     (effects (font (size 1.27 1.27)) (justify left bottom))
   )
-  (label "NET2_MX2+" (at 152.4 87.63 0) (fields_autoplaced)
+  (label "NET2_MX2+" (at 152.4 90.17 0) (fields_autoplaced)
     (effects (font (size 1.27 1.27)) (justify left bottom))
   )
@@
     (effects (font (size 1.27 1.27)) (justify left bottom))
   )
-  (label "NET2_MX2-" (at 152.4 85.09 0) (fields_autoplaced)
+  (label "NET2_MX2-" (at 152.4 87.63 0) (fields_autoplaced)
     (effects (font (size 1.27 1.27)) (justify left bottom))
   )
@@
     (effects (font (size 1.27 1.27)) (justify left bottom))
   )
-  (label "NET2_MX1-" (at 152.4 90.17 0) (fields_autoplaced)
+  (label "NET2_MX1-" (at 152.4 85.09 0) (fields_autoplaced)
     (effects (font (size 1.27 1.27)) (justify left bottom))
   )
@@
     (effects (font (size 1.27 1.27)) (justify left bottom))
   )
-  (label "NET1_MX2+" (at 152.4 59.69 0) (fields_autoplaced)
-    (effects (font (size 1.27 1.27)) (justify left bottom))
-  )
-  (label "NET1_MX1-" (at 152.4 62.23 0) (fields_autoplaced)
+  (label "NET1_MX2+" (at 152.4 62.23 0) (fields_autoplaced)
+    (effects (font (size 1.27 1.27)) (justify left bottom))
+  )
+  (label "NET1_MX1-" (at 152.4 57.15 0) (fields_autoplaced)
     (effects (font (size 1.27 1.27)) (justify left bottom))
   )
@@
     (effects (font (size 1.27 1.27)) (justify left bottom))
   )
-  (label "NET1_MX2-" (at 152.4 57.15 0) (fields_autoplaced)
-    (effects (font (size 1.27 1.27)) (justify left bottom))
-  )
+  (label "NET1_MX2-" (at 152.4 59.69 0) (fields_autoplaced)
+    (effects (font (size 1.27 1.27)) (justify left bottom))
+  )

Commit message: PCB V0.2
Parts:
- removed C4, C5: 0.1uF, Capacitor_SMD:C_0402_1005Metric, symbol Device:C
- removed D3: LED_RED, LED_SMD:LED_0603_1608Metric, symbol Device:LED
- removed D4: LED_BLUE, LED_SMD:LED_0603_1608Metric, symbol Device:LED
- removed D5: LED_GREEN, LED_SMD:LED_0603_1608Metric, symbol Device:LED
- removed D6: LED_YELLOW, LED_SMD:LED_0603_1608Metric, symbol Device:LED
- removed J11: Connect_J11, Connector_Hirose:Hirose_DF13C_CL535-0408-9-51_1x08-1MP_P1.25mm_Vertical, symbol Connector_Generic:Conn_01x08
- removed J15: IF_Xilinx14P, Connector_IDC:IDC-Header_2x07_P2.54mm_Vertical, symbol Connector_Generic:Conn_02x07_Odd_Even
- removed J18: Logic_Any, Connector_IDC:IDC-Header_2x05_P2.54mm_Horizontal, symbol Connector_Generic:Conn_02x05_Odd_Even
- removed J6: IF_Altera10P_2P00, Connector_PinHeader_2.00mm:PinHeader_2x05_P2.00mm_Vertical, symbol Connector_Generic:Conn_02x05_Odd_Even
- removed J7: Connect_J7, Connector_Hirose:Hirose_DF13C_CL535-0406-3-51_1x06-1MP_P1.25mm_Vertical, symbol Connector_Generic:Conn_01x06
- removed J8: IF_Altera10P_2P54, Connector_IDC:IDC-Header_2x05_P2.54mm_Vertical, symbol Connector_Generic:Conn_02x05_Odd_Even
- removed JP1, JP20, JP21: SolderJumper_3_Bridged12, Jumper:SolderJumper-3_P1.3mm_Bridged12_RoundedPad1.0x1.5mm, symbol Jumper:SolderJumper_3_Bridged12
- removed JP7: SolderJumper_2_Bridged, Jumper:SolderJumper-2_P1.3mm_Bridged_RoundedPad1.0x1.5mm, symbol Jumper:SolderJumper_2_Bridged
- removed JP8, JP9: SolderJumper_2_Open, Jumper:SolderJumper-2_P1.3mm_Open_RoundedPad1.0x1.5mm, symbol Jumper:SolderJumper_2_Open
- removed R1: 10k, Resistor_SMD:R_0402_1005Metric, symbol Device:R
- removed R2, R4: 5.1k, Resistor_SMD:R_0402_1005Metric, symbol Device:R
- removed R3: 47k, Resistor_SMD:R_0402_1005Metric, symbol Device:R
- removed U2, U3: SN74AVC4T245PW, Package_SO:TSSOP-16_4.4x5mm_P0.65mm, symbol Logic_LevelTranslator:SN74AVC4T245PW
- added J6: Connect_J14, Connector_PinSocket_2.54mm:PinSocket_1x02_P2.54mm_Horizontal, symbol Connector_Generic:Conn_01x02
- added JP1: SolderJumper_3_Open, Jumper:SolderJumper-3_P1.3mm_Open_RoundedPad1.0x1.5mm, symbol Jumper:SolderJumper_3_Open
- R12: value 5.1 -> 5.1k
Connections:
- net GND: now also U5.3 (2DIR); no longer U4.3 (2DIR)
- net J12_1: now also J6.2 (Pin_2)
- net J12_2: now also J6.1 (Pin_1)
- net J12_3: now also U5.6 (2A1); no longer U5.7 (2A2)
- net J12_6: now also U4.7 (2A2); no longer U5.3 (2DIR)
- net J12_7: now also U4.5 (1A2); no longer U4.6 (2A1)
- net J12_8: now also U4.4 (1A1); no longer U4.5 (1A2)
- net J12_9: now also U4.3 (2DIR); no longer U4.4 (1A1)
- net J13_2: now also U5.7 (2A2); no longer U4.7 (2A2)
- net SRST: now also JP15.2 (B); no longer JP11.2 (B)
- net TCK: now also JP12.2 (B); no longer JP15.2 (B)
- net TDI: now also JP11.2 (B); no longer JP12.2 (B)
- net TDO: now also JP16.2 (B); no longer JP13.2 (B)
- net TMS: now also JP13.2 (B); no longer JP17.2 (B)
- net TXD: now also JP17.2 (B); no longer JP16.2 (B)
- net VRef_D: now also JP1.2 (C)
- net ZYNQ7_3V3: now also JP1.1 (A)
- net ZYNQ7_5V: now also JP1.3 (B)
- net at U5.10 (2B2): now also JP14.1 (A); no longer JP17.1 (A)
- net at U5.11 (2B1): now also JP16.1 (A)
- net at U5.12 (1B2): now also JP17.1 (A); no longer JP16.1 (A)
- net at JP13.1 (A): now also U4.10 (2B2); no longer U4.11 (2B1)
- no-connect marks 8 -> 3
Other:
- moved on the sheet: C2, C3, JP13, JP14, JP16, JP17
